File: LeandroMedus/SWITCH_ENVELOPE.sch (KiCad schematic (older format))
At the start: 6 parts, among them U1 LTC5507, U2 74HCT4053, X1 XTAL

Commit message: Fin clase 2 faltante
Parts:
- C4: renamed from C1; footprint (none) -> OpenQCM:C_0805_HandSoldering
- C5: renamed from C2; footprint (none) -> OpenQCM:C_0805_HandSoldering
- C6: renamed from C3; footprint (none) -> OpenQCM:C_0805_HandSoldering
- U2: renamed from U1; footprint (none) -> OpenQCM:SOT-23-6
- U3: renamed from U2; footprint (none) -> OpenQCM:TSSOP16
- X1: footprint (none) -> OpenQCM:XTAL_con
Connections:
- net XTAL_IN is gone; now on net XTAL_N: X1.2
Changed lines of the file:
@@
 SWITCH_IN+
 $Comp
-L LTC5507 U1
+L LTC5507 U2
 U 1 1 56F94189
 P 5050 4500
-F 0 "U1" H 5250 4750 60  0000 C CNN
+F 0 "U2" H 5250 4750 60  0000 C CNN
 F 1 "LTC5507" H 5100 4100 60  0000 C CNN
-F 2 "" H 4950 4500 60  0000 C CNN
+F 2 "OpenQCM:SOT-23-6" H 4950 4500 60  0001 C CNN
 F 3 "" H 4950 4500 60  0000 C CNN
 	1    5050 4500
@@
 $EndComp
 $Comp
-L GND #PWR1
+L GND #PWR015
 U 1 1 56F944A1
 P 4250 4650
-F 0 "#PWR1" H 4250 4400 50  0001 C CNN
+F 0 "#PWR015" H 4250 4400 50  0001 C CNN
 F 1 "GND" H 4250 4500 50  0000 C CNN
 F 2 "" H 4250 4650 60  0000 C CNN
@@
 	4250 4550 4650 4550
 $Comp
-L +3V3 #PWR2
+L +3V3 #PWR016
 U 1 1 56F944BF
 P 4350 4200
-F 0 "#PWR2" H 4350 4050 50  0001 C CNN
+F 0 "#PWR016" H 4350 4050 50  0001 C CNN
 F 1 "+3V3" H 4350 4340 50  0000 C CNN
 F 2 "" H 4350 4200 60  0000 C CNN
@@
 	4350 4400 4650 4400
 $Comp
-L +3V3 #PWR3
+L +3V3 #PWR017
 U 1 1 56F944F4
 P 6650 4600
-F 0 "#PWR3" H 6650 4450 50  0001 C CNN
+F 0 "#PWR017" H 6650 4450 50  0001 C CNN
 F 1 "+3V3" H 6650 4740 50  0000 C CNN
 F 2 "" H 6650 4600 60  0000 C CNN
@@
 	5550 4700 6650 4700
 $Comp
-L Capacitor_SMD_HandSoldering C2
+L Capacitor_SMD_HandSoldering C5
 U 1 1 56F9450F
 P 5950 4550
-F 0 "C2" H 5950 4700 60  0000 C CNN
+F 0 "C5" H 5950 4700 60  0000 C CNN
 F 1 "pF" H 6100 4450 60  0000 C CNN
-F 2 "" H 5950 4550 60  0000 C CNN
+F 2 "OpenQCM:C_0805_HandSoldering" H 5950 4550 60  0001 C CNN
 F 3 "" H 5950 4550 60  0000 C CNN
 	1    5950 4550
@@
 	5700 4550 5550 4550
 $Comp
-L Capacitor_SMD_HandSoldering C1
+L Capacitor_SMD_HandSoldering C4
 U 1 1 56F94616
 P 5700 3900
-F 0 "C1" V 5700 4050 60  0000 C CNN
+F 0 "C4" V 5700 4050 60  0000 C CNN
 F 1 "pF" V 5800 4050 60  0000 C CNN
-F 2 "" H 5700 3900 60  0000 C CNN
+F 2 "OpenQCM:C_0805_HandSoldering" H 5700 3900 60  0001 C CNN
 F 3 "" H 5700 3900 60  0000 C CNN
 	1    5700 3900
@@
 $EndComp
 Wire Wire Line
-	5550 4400 5700 4400
-Wire Wire Line
-	5700 4400 5700 4150
-$Comp
-L 74HCT4053 U2
+	5700 4400 5550 4400
+Wire Wire Line
+	5700 4150 5700 4400
+$Comp
+L 74HCT4053 U3
 U 1 1 56F946CB
 P 7550 2500
-F 0 "U2" H 7550 3000 60  0000 C CNN
+F 0 "U3" H 7550 3000 60  0000 C CNN
 F 1 "74HCT4053" H 7550 2000 60  0000 C CNN
-F 2 "" H 7550 2550 60  0000 C CNN
+F 2 "OpenQCM:TSSOP16" H 7550 2550 60  0001 C CNN
 F 3 "" H 7550 2550 60  0000 C CNN
 	1    7550 2500
@@
 	7000 1650 7000 2100
 $Comp
-L GND #PWR4
+L GND #PWR018
 U 1 1 56F948B8
 P 6800 1750
-F 0 "#PWR4" H 6800 1500 50  0001 C CNN
+F 0 "#PWR018" H 6800 1500 50  0001 C CNN
 F 1 "GND" H 6800 1600 50  0000 C CNN
 F 2 "" H 6800 1750 60  0000 C CNN
@@
 	6800 1650 7000 1650
 $Comp
-L Capacitor_SMD_HandSoldering C3
+L Capacitor_SMD_HandSoldering C6
 U 1 1 56F94937
 P 8650 1800
-F 0 "C3" V 8650 1950 60  0000 C CNN
+F 0 "C6" V 8650 1950 60  0000 C CNN
 F 1 "pF" V 8750 1950 60  0000 C CNN
-F 2 "" H 8650 1800 60  0000 C CNN
+F 2 "OpenQCM:C_0805_HandSoldering" H 8650 1800 60  0001 C CNN
 F 3 "" H 8650 1800 60  0000 C CNN
 	1    8650 1800
@@
 $EndComp
 $Comp
-L GND #PWR8
+L GND #PWR019
 U 1 1 56F94A08
 P 8650 2200
-F 0 "#PWR8" H 8650 1950 50  0001 C CNN
+F 0 "#PWR019" H 8650 1950 50  0001 C CNN
 F 1 "GND" H 8650 2050 50  0000 C CNN
 F 2 "" H 8650 2200 60  0000 C CNN
@@
 	8650 2050 8650 2200
 $Comp
-L +3V3 #PWR7
+L +3V3 #PWR020
 U 1 1 56F94AF9
 P 8650 1350
-F 0 "#PWR7" H 8650 1200 50  0001 C CNN
+F 0 "#PWR020" H 8650 1200 50  0001 C CNN
 F 1 "+3V3" H 8650 1490 50  0000 C CNN
 F 2 "" H 8650 1350 60  0000 C CNN
@@
 	8400 2200 8400 2450
 $Comp
-L GND #PWR6
+L GND #PWR021
 U 1 1 56F94BAA
 P 8400 2450
-F 0 "#PWR6" H 8400 2200 50  0001 C CNN
+F 0 "#PWR021" H 8400 2200 50  0001 C CNN
 F 1 "GND" H 8400 2300 50  0000 C CNN
 F 2 "" H 8400 2450 60  0000 C CNN
@@
 Connection ~ 8200 2700
 $Comp
-L GND #PWR5
+L GND #PWR022
 U 1 1 56F94CE9
 P 8200 2850
-F 0 "#PWR5" H 8200 2600 50  0001 C CNN
+F 0 "#PWR022" H 8200 2600 50  0001 C CNN
 F 1 "GND" H 8200 2700 50  0000 C CNN
 F 2 "" H 8200 2850 60  0000 C CNN
@@
 F 0 "X1" H 3650 2100 60  0000 C CNN
 F 1 "XTAL" H 3650 1900 60  0000 C CNN
-F 2 "" H 3650 2000 60  0000 C CNN
+F 2 "OpenQCM:XTAL_con" H 3650 2000 60  0001 C CNN
 F 3 "" H 3650 2000 60  0000 C CNN
 	1    3650 2000
@@
 XTAL_P
 Text Label 3650 2650 1    60   ~ 0
-XTAL_IN
+XTAL_N
 Wire Notes Line
 	3150 1250 4000 1250
@@
 Text Notes 3200 1200 0    60   ~ 0
 Crystal
+Wire Wire Line
+	6200 4150 6200 4250
+Wire Wire Line
+	6200 4250 5700 4250
+Connection ~ 5700 4250
+Wire Wire Line
+	5650 4550 5650 5050
+Wire Wire Line
+	5650 5050 5900 5050
+Wire Wire Line
+	5900 5050 5900 5000
+Connection ~ 5650 4550
+$Comp
+L PWR_FLAG #FLG023
+U 1 1 56F96791
+P 5900 5000
+F 0 "#FLG023" H 5900 5095 50  0001 C CNN
+F 1 "PWR_FLAG" H 5900 5180 50  0000 C CNN
+F 2 "" H 5900 5000 60  0000 C CNN
+F 3 "" H 5900 5000 60  0000 C CNN
+	1    5900 5000
+	1    0    0    -1
+$EndComp
+$Comp
+L PWR_FLAG #FLG024
+U 1 1 56F9668A
+P 6200 4150
+F 0 "#FLG024" H 6200 4245 50  0001 C CNN
+F 1 "PWR_FLAG" H 6200 4330 50  0000 C CNN
+F 2 "" H 6200 4150 60  0000 C CNN
+F 3 "" H 6200 4150 60  0000 C CNN
+	1    6200 4150
+	1    0    0    -1
+$EndComp
 $EndSCHEMATC
