File: JuanCruz_GL/Re_intento/Ejercicio_2.kicad_pcb (KiCad board)
At the start: 2 copper layers, 38.7 x 31.4 mm, 17 parts, among them P1 CONN_01X14, P2 CONN_01X14, U1 SN74LVC1GX04, U2 74HCT4053, U3 LTC5507, X1 XTAL

Commit message: Ejercicio 3 JCGL
Parts:
- G***: moved to B.Cu
- moved C6 76.0 mm to (145.0, 104.3), turned to 90 degrees
- moved U2 68.7 mm to (141.3, 103.7), turned to 270 degrees
- moved C4 59.7 mm to (140.7, 109.2)
- moved U3 53.8 mm to (164.3, 106.9), turned to 270 degrees
- moved C5 48.4 mm to (164.7, 102.1)
- moved C3 48.1 mm to (164.7, 100.3)
- moved C2 46.1 mm to (149.4, 101.2), turned to 90 degrees
- moved U1 43.9 mm to (160.1, 101.3), turned to 270 degrees
- moved R3 42.6 mm to (154.1, 108.7)
- moved C1 42.5 mm to (146.8, 101.2), turned to 270 degrees
- moved R2 32.9 mm to (148.0, 108.7), turned to 180 degrees
- moved R1 28.4 mm to (160.2, 105.9), turned to 180 degrees
- moved PTC1 20.5 mm to (160.2, 108.7)
- moved G*** 1.16 mm to (152.1, 105.2)
Routing:
- net GND: track 0.00 -> 92.2 mm, vias 0 -> 6
- net /SWITCH_ENVELOPE/xtal_P: track 0.00 -> 39.1 mm, vias 0 -> 1
- net /SWITCH_ENVELOPE/xtal_N: track 0.00 -> 39.1 mm, vias 0 -> 1
- net /OSC_DRIVER/Switch_IN+: track 0.00 -> 29.3 mm
- net +3V3: track 0.00 -> 28.9 mm, vias 0 -> 2
- net Net-(C4-Pad2): track 0.00 -> 24.0 mm, vias 0 -> 2
- net /OSC_DRIVER/Switch_IN-: track 0.00 -> 23.5 mm, vias 0 -> 2
- net Net-(R2-Pad1): track 0.00 -> 19.9 mm
- net +5V: track 0.00 -> 16.5 mm, vias 0 -> 2
- net /Arduino/FREQUENCY_IN: track 0.00 -> 12.9 mm, vias 0 -> 2
- net /Arduino/ENVELOPE_IN: track 0.00 -> 12.6 mm, vias 0 -> 2
- net /Arduino/DIG_CONTROL: track 0.00 -> 8.85 mm, vias 0 -> 2
- net Net-(C5-Pad2): track 0.00 -> 7.22 mm
- net /Arduino/PTC: track 0.00 -> 6.96 mm
- net Net-(C4-Pad1): track 0.00 -> 3.16 mm
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- added copper zone on B.Cu, net GND
- added copper zone on F.Cu, net GND
Other:
- net class Default: trace_width 0.2032 -> 0.2; via_dia 0.6 -> 0.5
- net class Diff added: clearance 0.2, trace_width 0.2, via_dia 0.3, via_drill 0.25
- net class PW: trace_width 0.5 -> 0.2; via_dia 0.6 -> 0.3; via_drill 0.4 -> 0.25
- rule trace_min: 0.2032 -> 0.2
- rule via_min_drill: 0.3 -> 0.25
- rule via_min_size: 0.4 -> 0.3
- board text added: "UNER Ki-CAD"
