File: christianhalter/SWITCH.sch (KiCad schematic (older format))
At the start: 6 parts, among them U2 74HCT4053, X1 XTAL

Commit message: componente nuevo
Parts:
- C4: renamed from C1; footprint (none) -> halter:C_0805_HandSoldering
- C5: renamed from C2; footprint (none) -> halter:C_0805_HandSoldering
- C6: renamed from C3; footprint (none) -> halter:C_0805_HandSoldering
- U2: footprint (none) -> halter:TSSOP16
- U3: renamed from U?; footprint (none) -> halter:SOT-23-6
- X1: footprint (none) -> halter:XTAL_con
Changed lines of the file:
@@
 ENVELOPE_OUT
 $Comp
-L +3V3 #PWR2
+L +3V3 #PWR015
 U 1 1 56F93E0D
 P 4150 3550
-F 0 "#PWR2" H 4150 3400 50  0001 C CNN
+F 0 "#PWR015" H 4150 3400 50  0001 C CNN
 F 1 "+3V3" H 4150 3690 50  0000 C CNN
 F 2 "" H 4150 3550 60  0000 C CNN
@@
 	4150 3700 4150 3550
 $Comp
-L GND #PWR1
+L GND #PWR016
 U 1 1 56F93E2E
 P 3950 3850
-F 0 "#PWR1" H 3950 3600 50  0001 C CNN
+F 0 "#PWR016" H 3950 3600 50  0001 C CNN
 F 1 "GND" H 3950 3700 50  0000 C CNN
 F 2 "" H 3950 3850 60  0000 C CNN
@@
 F 0 "U2" H 7350 2450 60  0000 C CNN
 F 1 "74HCT4053" H 7350 1450 60  0000 C CNN
-F 2 "" H 7350 2000 60  0000 C CNN
+F 2 "halter:TSSOP16" H 7350 2000 60  0001 C CNN
 F 3 "" H 7350 2000 60  0000 C CNN
 	1    7350 1950
@@
 $EndComp
 $Comp
-L GND #PWR4
+L GND #PWR017
 U 1 1 56F93FE4
 P 6600 1350
-F 0 "#PWR4" H 6600 1100 50  0001 C CNN
+F 0 "#PWR017" H 6600 1100 50  0001 C CNN
 F 1 "GND" H 6600 1200 50  0000 C CNN
 F 2 "" H 6600 1350 60  0000 C CNN
@@
 $EndComp
 $Comp
-L GND #PWR6
+L GND #PWR018
 U 1 1 56F93FFE
 P 8000 2350
-F 0 "#PWR6" H 8000 2100 50  0001 C CNN
+F 0 "#PWR018" H 8000 2100 50  0001 C CNN
 F 1 "GND" H 8000 2200 50  0000 C CNN
 F 2 "" H 8000 2350 60  0000 C CNN
@@
 $EndComp
 $Comp
-L GND #PWR8
+L GND #PWR019
 U 1 1 56F94016
 P 8850 2000
-F 0 "#PWR8" H 8850 1750 50  0001 C CNN
+F 0 "#PWR019" H 8850 1750 50  0001 C CNN
 F 1 "GND" H 8850 1850 50  0000 C CNN
 F 2 "" H 8850 2000 60  0000 C CNN
@@
 $EndComp
 $Comp
-L GND #PWR5
+L GND #PWR020
 U 1 1 56F94058
 P 8000 1850
-F 0 "#PWR5" H 8000 1600 50  0001 C CNN
+F 0 "#PWR020" H 8000 1600 50  0001 C CNN
 F 1 "GND" H 8000 1700 50  0000 C CNN
 F 2 "" H 8000 1850 60  0000 C CNN
@@
 $EndComp
 $Comp
-L +5V #PWR7
+L +5V #PWR021
 U 1 1 56F94070
 P 8850 1450
-F 0 "#PWR7" H 8850 1300 50  0001 C CNN
+F 0 "#PWR021" H 8850 1300 50  0001 C CNN
 F 1 "+5V" H 8850 1590 50  0000 C CNN
 F 2 "" H 8850 1450 60  0000 C CNN
@@
 $EndComp
 $Comp
-L +3V3 #PWR3
+L +3V3 #PWR022
 U 1 1 56F940B8
 P 6400 3800
-F 0 "#PWR3" H 6400 3650 50  0001 C CNN
+F 0 "#PWR022" H 6400 3650 50  0001 C CNN
 F 1 "+3V3" H 6400 3940 50  0000 C CNN
 F 2 "" H 6400 3800 60  0000 C CNN
@@
 F 0 "X1" H 4900 2200 60  0000 C CNN
 F 1 "XTAL" H 4900 2000 60  0000 C CNN
-F 2 "" H 4900 2100 60  0000 C CNN
+F 2 "halter:XTAL_con" H 4900 2100 60  0001 C CNN
 F 3 "" H 4900 2100 60  0000 C CNN
 	1    4900 2100
@@
 $EndComp
 $Comp
-L Capacitor_SMD_HandSoldering C2
+L Capacitor_SMD_HandSoldering C5
 U 1 1 56F9428F
 P 5900 3850
-F 0 "C2" H 5900 4000 60  0000 C CNN
+F 0 "C5" H 5900 4000 60  0000 C CNN
 F 1 "pF" H 6000 3700 60  0000 C CNN
-F 2 "" H 5900 3850 60  0000 C CNN
+F 2 "halter:C_0805_HandSoldering" H 5900 3850 60  0001 C CNN
 F 3 "" H 5900 3850 60  0000 C CNN
 	1    5900 3850
@@
 $EndComp
 $Comp
-L Capacitor_SMD_HandSoldering C1
+L Capacitor_SMD_HandSoldering C4
 U 1 1 56F9434C
 P 5800 3250
-F 0 "C1" H 5800 3400 60  0000 C CNN
+F 0 "C4" H 5800 3400 60  0000 C CNN
 F 1 "pF" H 5900 3100 60  0000 C CNN
-F 2 "" H 5800 3250 60  0000 C CNN
+F 2 "halter:C_0805_HandSoldering" H 5800 3250 60  0001 C CNN
 F 3 "" H 5800 3250 60  0000 C CNN
 	1    5800 3250
@@
 $EndComp
 $Comp
-L Capacitor_SMD_HandSoldering C3
+L Capacitor_SMD_HandSoldering C6
 U 1 1 56F943E7
 P 8850 1750
-F 0 "C3" H 8850 1900 60  0000 C CNN
+F 0 "C6" H 8850 1900 60  0000 C CNN
 F 1 "100nF" H 8950 1600 60  0000 C CNN
-F 2 "" H 8850 1750 60  0000 C CNN
+F 2 "halter:C_0805_HandSoldering" H 8850 1750 60  0001 C CNN
 F 3 "" H 8850 1750 60  0000 C CNN
 	1    8850 1750
@@
 Wire Wire Line
 	8500 1450 8850 1450
-Wire Wire Line
-	6600 1350 6850 1350
-Wire Wire Line
-	6850 1350 6850 1550
 Wire Wire Line
 	6600 1650 6850 1650
@@
 	5800 2150 5800 3000
 Wire Wire Line
-	5800 3700 5800 3500
-Wire Wire Line
 	6400 4000 6400 3800
 Wire Wire Line
@@
 Connection ~ 6400 3850
 $Comp
-L LTC5507 U?
+L LTC5507 U3
 U 1 1 56F95CB0
 P 4900 3850
-F 0 "U?" H 4900 4200 60  0000 C CNN
+F 0 "U3" H 4900 4200 60  0000 C CNN
 F 1 "LTC5507" H 4900 3400 60  0000 C CNN
-F 2 "" H 5800 3700 60  0000 C CNN
+F 2 "halter:SOT-23-6" H 5800 3700 60  0001 C CNN
 F 3 "" H 5800 3700 60  0000 C CNN
 	1    4900 3850
@@
 	5800 3700 5550 3700
 Wire Wire Line
-	5650 3850 5550 3850
-Wire Wire Line
 	6400 4000 5550 4000
+Wire Wire Line
+	5800 3700 5800 3500
+Wire Wire Line
+	5550 3850 5650 3850
+Wire Wire Line
+	6600 1350 6850 1350
+Wire Wire Line
+	6850 1350 6850 1550
+$Comp
+L PWR_FLAG #FLG023
+U 1 1 56F96781
+P 5600 3650
+F 0 "#FLG023" H 5600 3745 50  0001 C CNN
+F 1 "PWR_FLAG" H 5600 3830 50  0000 C CNN
+F 2 "" H 5600 3650 60  0000 C CNN
+F 3 "" H 5600 3650 60  0000 C CNN
+	1    5600 3650
+	1    0    0    -1
+$EndComp
+Wire Wire Line
+	5600 3650 5600 3700
+Connection ~ 5600 3700
+$Comp
+L PWR_FLAG #FLG024
+U 1 1 56F968DE
+P 5600 4150
+F 0 "#FLG024" H 5600 4245 50  0001 C CNN
+F 1 "PWR_FLAG" H 5600 4330 50  0000 C CNN
+F 2 "" H 5600 4150 60  0000 C CNN
+F 3 "" H 5600 4150 60  0000 C CNN
+	1    5600 4150
+	-1   0    0    1
+$EndComp
+Wire Wire Line
+	5600 4150 5600 3850
+Connection ~ 5600 3850
 $EndSCHEMATC

Commit message: Gerber
Parts:
- C4, C5, C6: footprint halter:C_0805_HandSoldering -> halter:C_0603_HandSoldering
Changed lines of the file:
@@
 F 0 "C5" H 5900 4000 60  0000 C CNN
 F 1 "pF" H 6000 3700 60  0000 C CNN
-F 2 "halter:C_0805_HandSoldering" H 5900 3850 60  0001 C CNN
+F 2 "halter:C_0603_HandSoldering" H 5900 3850 60  0001 C CNN
 F 3 "" H 5900 3850 60  0000 C CNN
 	1    5900 3850
@@
 F 0 "C4" H 5800 3400 60  0000 C CNN
 F 1 "pF" H 5900 3100 60  0000 C CNN
-F 2 "halter:C_0805_HandSoldering" H 5800 3250 60  0001 C CNN
+F 2 "halter:C_0603_HandSoldering" H 5800 3250 60  0001 C CNN
 F 3 "" H 5800 3250 60  0000 C CNN
 	1    5800 3250
@@
 F 0 "C6" H 8850 1900 60  0000 C CNN
 F 1 "100nF" H 8950 1600 60  0000 C CNN
-F 2 "halter:C_0805_HandSoldering" H 8850 1750 60  0001 C CNN
+F 2 "halter:C_0603_HandSoldering" H 8850 1750 60  0001 C CNN
 F 3 "" H 8850 1750 60  0000 C CNN
 	1    8850 1750

Commit message: Libreria nueva
Connections:
- net Switch_IN+ renamed CON2
- net Switch_IN- renamed CON1
Changed lines of the file:
@@
 LIBS:XTAL_SMD_HandSoldering
 LIBS:ltc5507
+LIBS:74hct4053_pringle
 LIBS:halter-cache
 EELAYER 25 0
@@
 Comment4 ""
 $EndDescr
-Text HLabel 6700 2250 0    60   Input ~ 0
-Switch_IN+
-Text HLabel 6600 1650 0    60   Input ~ 0
-Switch_IN-
 Text HLabel 7950 2150 2    60   Input ~ 0
 DIG_CONTROL
@@
 	1    0    0    -1
 $EndComp
-Wire Wire Line
-	4150 3700 4150 3550
 $Comp
 L GND #PWR016
@@
 F 3 "" H 3950 3850 60  0000 C CNN
 	1    3950 3850
-	1    0    0    -1
-$EndComp
-Wire Wire Line
-	4250 4350 3000 4350
-$Comp
-L 74HCT4053 U2
-U 1 1 56F93E7F
-P 7350 1950
-F 0 "U2" H 7350 2450 60  0000 C CNN
-F 1 "74HCT4053" H 7350 1450 60  0000 C CNN
-F 2 "halter:TSSOP16" H 7350 2000 60  0001 C CNN
-F 3 "" H 7350 2000 60  0000 C CNN
-	1    7350 1950
 	1    0    0    -1
 $EndComp
@@
 	0    1    1    0
 $EndComp
-Wire Wire Line
-	8850 1450 8850 1500
-Wire Wire Line
-	7850 1550 8500 1550
-Wire Wire Line
-	8500 1550 8500 1450
-Wire Wire Line
-	8500 1450 8850 1450
-Wire Wire Line
-	6600 1650 6850 1650
 Text Label 4900 1900 0    60   ~ 0
 xtal_P
@@
 Text Label 6100 2350 2    60   ~ 0
 xtal_N
-Wire Wire Line
-	6000 1750 6850 1750
-Wire Wire Line
-	6850 2350 6100 2350
-Wire Wire Line
-	6700 2250 6850 2250
-Wire Wire Line
-	7850 2250 8000 2250
-Wire Wire Line
-	8000 2250 8000 2350
-Wire Wire Line
-	8000 1850 7850 1850
-Wire Wire Line
-	7850 1650 8000 1650
-Wire Wire Line
-	8000 1650 8000 1850
-Wire Wire Line
-	7850 1750 8000 1750
-Connection ~ 8000 1750
 NoConn ~ 6850 1850
 NoConn ~ 6850 1950
 NoConn ~ 6850 2050
-Wire Wire Line
-	7850 2150 7950 2150
-Wire Wire Line
-	7850 2050 7900 2050
-Wire Wire Line
-	7900 2050 7900 2150
-Connection ~ 7900 2150
-Wire Wire Line
-	6850 2150 5800 2150
-Wire Wire Line
-	5800 2150 5800 3000
-Wire Wire Line
-	6400 4000 6400 3800
-Wire Wire Line
-	6150 3850 6400 3850
-Connection ~ 6400 3850
 $Comp
 L LTC5507 U3
@@
 	1    0    0    -1
 $EndComp
-Wire Wire Line
-	3950 3850 4250 3850
-Wire Wire Line
-	4150 3700 4250 3700
-Wire Wire Line
-	4250 4350 4250 4000
-Wire Wire Line
-	5800 3700 5550 3700
-Wire Wire Line
-	6400 4000 5550 4000
-Wire Wire Line
-	5800 3700 5800 3500
-Wire Wire Line
-	5550 3850 5650 3850
-Wire Wire Line
-	6600 1350 6850 1350
-Wire Wire Line
-	6850 1350 6850 1550
 $Comp
 L PWR_FLAG #FLG023
@@
 	1    0    0    -1
 $EndComp
-Wire Wire Line
-	5600 3650 5600 3700
-Connection ~ 5600 3700
 $Comp
 L PWR_FLAG #FLG024
@@
 $EndComp
 Wire Wire Line
+	4150 3700 4150 3550
+Wire Wire Line
+	4250 4350 3000 4350
+Wire Wire Line
+	8850 1450 8850 1500
+Wire Wire Line
+	7850 1550 8500 1550
+Wire Wire Line
+	8500 1550 8500 1450
+Wire Wire Line
+	8500 1450 8850 1450
+Wire Wire Line
+	6600 1650 6850 1650
+Wire Wire Line
+	6000 1750 6850 1750
+Wire Wire Line
+	6850 2350 6100 2350
+Wire Wire Line
+	7850 2250 8000 2250
+Wire Wire Line
+	8000 2250 8000 2350
+Wire Wire Line
+	8000 1850 7850 1850
+Wire Wire Line
+	7850 1650 8000 1650
+Wire Wire Line
+	8000 1650 8000 1850
+Wire Wire Line
+	7850 1750 8000 1750
+Connection ~ 8000 1750
+Wire Wire Line
+	7850 2150 7950 2150
+Wire Wire Line
+	7850 2050 7900 2050
+Wire Wire Line
+	7900 2050 7900 2150
+Connection ~ 7900 2150
+Wire Wire Line
+	6850 2150 5800 2150
+Wire Wire Line
+	5800 2150 5800 3000
+Wire Wire Line
+	6400 4000 6400 3800
+Wire Wire Line
+	6150 3850 6400 3850
+Connection ~ 6400 3850
+Wire Wire Line
+	3950 3850 4250 3850
+Wire Wire Line
+	4150 3700 4250 3700
+Wire Wire Line
+	4250 4350 4250 4000
+Wire Wire Line
+	5800 3700 5550 3700
+Wire Wire Line
+	6400 4000 5550 4000
+Wire Wire Line
+	5800 3700 5800 3500
+Wire Wire Line
+	5550 3850 5650 3850
+Wire Wire Line
+	6600 1350 6850 1350
+Wire Wire Line
+	6850 1350 6850 1550
+Wire Wire Line
+	5600 3650 5600 3700
+Connection ~ 5600 3700
+Wire Wire Line
 	5600 4150 5600 3850
 Connection ~ 5600 3850
+Text HLabel 5900 1000 0    60   Input ~ 0
+CON[1..2]
+Wire Bus Line
+	5900 1000 6500 1000
+Text Label 6600 1650 0    60   ~ 0
+CON1
+Wire Wire Line
+	6850 2250 6600 2250
+Text Label 6600 2250 0    60   ~ 0
+CON2
+Wire Bus Line
+	6500 1000 6500 2100
+Entry Bus Bus
+	6500 2100 6600 2200
+Wire Wire Line
+	6600 2250 6600 2200
+Entry Bus Bus
+	6500 1550 6600 1650
+$Comp
+L 74HCT4053 U2
+U 1 1 56F93E7F
+P 7350 1950
+F 0 "U2" H 7350 2450 60  0000 C CNN
+F 1 "74HCT4053" H 7350 1450 60  0000 C CNN
+F 2 "halter:TSSOP16" H 7350 2000 60  0001 C CNN
+F 3 "" H 7350 2000 60  0000 C CNN
+	1    7350 1950
+	1    0    0    -1
+$EndComp
 $EndSCHEMATC
