File: christianhalter/halter.sch (KiCad schematic (older format))
At the start: 0 parts

Commit message: Libreria nueva
Changed lines of the file:
@@
 LIBS:XTAL_SMD_HandSoldering
 LIBS:ltc5507
+LIBS:74hct4053_pringle
 LIBS:halter-cache
 EELAYER 25 0
@@
 F0 "SWITCH" 60
 F1 "SWITCH.sch" 60
-F2 "Switch_IN+" I R 8500 4800 60
-F3 "Switch_IN-" I R 8500 4350 60
-F4 "DIG_CONTROL" I L 5050 4550 60
-F5 "ENVELOPE_OUT" I L 5050 5000 60
+F2 "DIG_CONTROL" I L 5050 4550 60
+F3 "ENVELOPE_OUT" I L 5050 5000 60
+F4 "CON[1..2]" I R 8500 5250 60
 $EndSheet
 Wire Wire Line
@@
 Wire Wire Line
 	3950 5000 5050 5000
-Wire Wire Line
-	8500 4350 10200 4350
-Wire Wire Line
-	10200 4350 10200 2500
-Wire Wire Line
-	10200 2500 9950 2500
-Wire Wire Line
-	9950 2100 10450 2100
-Wire Wire Line
-	10450 2100 10450 4800
-Wire Wire Line
-	10450 4800 8500 4800
+Entry Wire Line
+	9950 2100 10050 2200
+Entry Wire Line
+	9950 2500 10050 2600
+Wire Bus Line
+	10050 2200 10050 4150
+Wire Bus Line
+	10050 4150 8650 4150
+Wire Bus Line
+	8650 4150 8650 5250
+Text Label 10050 3400 0    60   ~ 0
+CON[1..2]
+Text Label 10000 2150 0    60   ~ 0
+CON1
+Text Label 10000 2550 0    60   ~ 0
+CON2
+Wire Bus Line
+	8650 5250 8500 5250
 $EndSCHEMATC
